File: Sharp_PC-2500/Sharp_PC-2500_RAM_Upgrade/Sharp_PC-2500_RAM_Upgrade.kicad_sch (KiCad schematic)
At the start: 4 parts, among them J2 FPC, U1 74HCT04, U2 62256

Commit message: Initial commit
Parts:
- added H1, H2: MountingHole, MountingHole:MountingHole_3.2mm_M3, symbol Mechanical:MountingHole
- added H3: MountingHole_Pad, MountingHole:MountingHole_3.2mm_M3_DIN965_Pad_TopBottom, symbol Mechanical:MountingHole_Pad
- J1: renamed from J2; footprint Connector_FFC-FPC:Amphenol_F32Q-1A7x1-11030_1x30-1MP_P0.5mm_Horizontal -> Sharp_PC-2500:Sharp PC-2500 30-pin TFC Connector
Connections:
- net GND: now also H3.1
Other:
- note removed: "WORK IN PROGRESS"
