File: Sharp_MZ-80B/Sharp_MZ-80B_New_Power_Supply/Sharp_MZ-80B_New_Power_Supply.kicad_sch (KiCad schematic)
At the start: 19 parts, among them J1 +12V (NS), J2 DC In, J3 To Tape Deck, J4 To Motherboard, U1 PSU5, U2 R-78CK5.0-0.5

Commit message: Revised PSU design
Parts:
- added D2: 1.5KE15A, Diode_THT:D_DO-201AE_P15.24mm_Horizontal, symbol Diode:1.5KExxA
- added F1: T4A, Fuse:Littelfuse_5x20mm, symbol Device:Fuse
- C1: value 4700µF -> 4700µF 25V; footprint Capacitor_THT:CP_Radial_D16.0mm_P7.50mm -> Capacitor_THT:CP_Axial_L40.0mm_D16.0mm_P48.00mm_Horizontal
- C2, C4, C6, C8: footprint Capacitor_THT:C_Disc_D3.8mm_W2.6mm_P2.50mm -> Capacitor_THT:C_Disc_D4.7mm_W2.5mm_P5.00mm
- J1: value +12V (NS) -> +12V (S)
- J2: footprint Clueless_Engineer:TJC1-2A -> Connector_JST:JST_VH_B2P-VH_1x02_P3.96mm_Vertical
- R1: value 2.2Ω -> 2.2Ω 2W
Connections:
- net +12V: now also J1.1 (Pin_1), J4.3 (Pin_3), D2.1 (A1), F1.2; no longer J2.2 (Pin_2), J3.3 (Pin_3), J4.4 (Pin_4)
- net +12V NS: now also J3.3 (Pin_3); no longer J1.1 (Pin_1)
- net +5V: now also J4.2 (Pin_2); no longer J4.3 (Pin_3)
- net -5V: now also J4.4 (Pin_4); no longer J4.2 (Pin_2)
- net GND: now also D2.2 (A2)
- new net +12V_{IN}: F1.1, J2.2 (Pin_2)
Other:
- moved on the sheet: J1, J2, J3, J4

Commit message: Revised DC input connector
Parts:
- J2: footprint Connector_JST:JST_VH_B2P-VH_1x02_P3.96mm_Vertical -> Clueless_Engineer:TJC1-2A
Changed lines of the file:
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@@
 			)
 		)
-		(property "Footprint" "Connector_JST:JST_VH_B2P-VH_1x02_P3.96mm_Vertical"
+		(property "Footprint" "Clueless_Engineer:TJC1-2A"
 			(at 25.4 74.93 0)
 			(hide yes)
