File: Sharp_MZ-80B/Sharp_MZ-CVBS/Sharp_MZ-80CVBS.kicad_pcb (KiCad board)
At the start: 2 copper layers, 79 x 47 mm, 33 parts, among them J1 VOLUME, J2 AUDIO OUT, J3 INPUT, J4 VIDEO OUT, Q1 2N3904, U1 74LS07, U2 LM386N-4, U3 LM7805

Commit message: Fixed 7805 silkscreen
Routing:
- added copper zone on F.Cu, net GND
Changed lines of the file:
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@@
 	)
 	(gr_rect
-		(start 92.0496 96.1456)
-		(end 102.2858 112.046)
+		(start 92.27201 96.425)
+		(end 102.05415 111.665)
 		(stroke
 			(width 0.1)
@@
 	)
 	(zone
+		(net "GND")
+		(layer "F.Cu")
+		(hatch edge 0.5)
+		(priority 1)
+		(connect_pads
+			(clearance 0.3)
+		)
+		(min_thickness 0.25)
+		(fill yes
+			(thermal_gap 0.5)
+			(thermal_bridge_width 0.5)
+			(smoothing fillet)
+			(radius 0.5)
+			(island_removal_mode 0)
+		)
+		(polygon
+			(pts
+				(xy 88.265 86.9) (xy 102.87 86.9) (xy 102.87 112.3) (xy 88.265 112.3)
+			)
+		)
+	)
+	(zone
